File: PCBs/PerceptronAdder/PerceptronAdder.kicad_pcb (KiCad board)
At the start: 2 copper layers, 122 x 132 mm, 60 parts, among them J1 Conn_02x10, J2 Conn_01x02_Pin

Commit message: Get rid of jlc silkscreen.
Other:
- board text removed: "jlcjlcjlcjlc"
Changed lines of the file:
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@@
 	(title_block
 		(title "Perceptron Adder")
-		(date "2026-02-07")
-		(rev "2")
+		(date "2026-02-20")
+		(rev "2.1")
 		(company "RDB64")
 	)
@@
 		)
 	)
-	(gr_text "Rev ${REVISION}, ${ISSUE_DATE}, ${COMPANY}"
-		(at 125.5 155 0)
-		(layer "F.SilkS")
-		(effects
-			(font
-				(size 1 1)
-				(thickness 0.1)
-			)
-			(justify bottom)
-		)
-	)
-	(gr_text "jlcjlcjlcjlc"
-		(at 77.5 154.5 0)
+	(gr_text "+"
+		(at 180 77.5 0)
 		(layer "B.SilkS")
 		(effects
 			(font
-				(size 1 1)
+				(size 1.2 1.2)
 				(thickness 0.1)
 			)
-			(justify right bottom mirror)
+			(justify mirror)
 		)
 	)
-	(gr_text "+"
-		(at 180 77.5 0)
+	(gr_text "-"
+		(at 180 87.5 0)
 		(layer "B.SilkS")
 		(effects
@@
 		)
 	)
-	(gr_text "-"
-		(at 180 87.5 0)
+	(gr_text "Rev ${REVISION}, ${ISSUE_DATE}, ${COMPANY}"
+		(at 66.5 134 270)
 		(layer "B.SilkS")
 		(effects
 			(font
-				(size 1.2 1.2)
+				(size 1 1)
 				(thickness 0.1)
 			)
-			(justify mirror)
+			(justify bottom mirror)
 		)
 	)
