File: PCBs/PerceptronAdder/PerceptronAdder.kicad_pcb (KiCad board)
At the start: 2 copper layers, 122 x 132 mm, 60 parts, among them J1 Conn_02x10, J2 Conn_01x02_Pin

Commit message: Added resistor values to silkscreen.
Parts:
- R1, R10, R11, R12, R13, R14, R15, R16, R17, R18, R19, R2, R20, R21, R22, R23, R24, R25, R26, R27, R28, R29, R3, R30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: footprint Resistor_THT:R_Axial_DIN0207_L6.3mm_D2.5mm_P7.62mm_Horizontal -> PerceptronAdderFootprints:R_Axial_DIN0207_L6.3mm_D2.5mm_P7.62mm_Horizontal
