File: PCBs/PerceptronAdder/PerceptronAdder.kicad_sch (KiCad schematic)
At the start: 80 parts, among them J1 Conn_02x10, J2 Conn_01x02_Pin, J3 Conn_01x02_Socket

Commit message: Get the right BoM fields
Parts:
- K1, K10, K11, K12, K13, K14, K15, K16, K17, K2, K3, K4, K5, K6, K7, K8, K9: value ~ -> 6mm
- RC1: value ~ -> 20P
Changed lines of the file:
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@@
 			)
 		)
-		(property "Value" "~"
+		(property "Value" "6mm"
 			(at 68.58 154.94 0)
 			(effects
@@
 			)
 		)
-		(property "Value" "~"
+		(property "Value" "6mm"
 			(at 72.39 185.42 0)
 			(effects
@@
 			)
 		)
-		(property "Value" "~"
+		(property "Value" "6mm"
 			(at 83.82 177.8 0)
 			(effects
@@
 			)
 		)
-		(property "Value" "~"
+		(property "Value" "6mm"
 			(at 76.2 154.94 0)
 			(effects
@@
 			)
 		)
-		(property "Value" "~"
+		(property "Value" "6mm"
 			(at 60.96 154.94 0)
 			(effects
@@
 			)
 		)
-		(property "Value" "~"
+		(property "Value" "6mm"
 			(at 83.82 162.56 0)
 			(effects
@@
 			)
 		)
-		(property "Value" "~"
+		(property "Value" "6mm"
 			(at 76.2 177.8 0)
 			(effects
@@
 			)
 		)
-		(property "Value" "~"
+		(property "Value" "20P"
 			(at 39.37 172.7199 0)
 			(effects
@@
 			)
 		)
-		(property "Value" "~"
+		(property "Value" "6mm"
 			(at 68.58 177.8 0)
 			(effects
@@
 			)
 		)
-		(property "Value" "~"
+		(property "Value" "6mm"
 			(at 76.2 170.18 0)
 			(effects
@@
 			)
 		)
-		(property "Value" "~"
+		(property "Value" "6mm"
 			(at 68.58 170.18 0)
 			(effects
@@
 			)
 		)
-		(property "Value" "~"
+		(property "Value" "6mm"
 			(at 83.82 170.18 0)
 			(effects
@@
 			)
 		)
-		(property "Value" "~"
+		(property "Value" "6mm"
 			(at 68.58 162.56 0)
 			(effects
@@
 			)
 		)
-		(property "Value" "~"
+		(property "Value" "6mm"
 			(at 60.96 170.18 0)
 			(effects
@@
 			)
 		)
-		(property "Value" "~"
+		(property "Value" "6mm"
 			(at 60.96 162.56 0)
 			(effects
@@
 			)
 		)
-		(property "Value" "~"
+		(property "Value" "6mm"
 			(at 60.96 177.8 0)
 			(effects
@@
 			)
 		)
-		(property "Value" "~"
+		(property "Value" "6mm"
 			(at 76.2 162.56 0)
 			(effects
@@
 			)
 		)
-		(property "Value" "~"
+		(property "Value" "6mm"
 			(at 83.82 154.94 0)
 			(effects

Commit message: Write the soldering section.
Parts:
- J1: Alt Link (none) -> https://www.digikey.com/en/products/detail/w%C3%BCrth-elekt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
Changed lines of the file:
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@@
 			)
 		)
-		(property "Alt Link" ""
+		(property "Alt Link" "https://www.digikey.com/en/products/detail/w%C3%BCrth-elektronik/61202021621/2060592"
 			(at 133.35 45.72 0)
 			(effects

Commit message: Get the right meters in the BoM, add a photo, and update that section to reflect these meters.
Parts:
- MES1: Alt Link (none) -> https://www.ebay.com/itm/172934983437; Link https://www.aliexpress.us/item/3256807093883789.html -> https://www.aliexpress.us/item/3256806998543963.html
Changed lines of the file:
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@@
 			)
 		)
-		(property "Link" "https://www.aliexpress.us/item/3256807093883789.html"
+		(property "Link" "https://www.aliexpress.us/item/3256806998543963.html"
 			(at 137.16 143.51 0)
 			(effects
@@
 			)
 		)
-		(property "Alt Link" ""
+		(property "Alt Link" "https://www.ebay.com/itm/172934983437"
 			(at 137.16 143.51 0)
 			(effects
