File: PCBs/PerceptronInput/PerceptronInput.kicad_sch (KiCad schematic)
At the start: 57 parts, among them J1 Conn_02x10, J2 Conn_01x04_Pin, J3 Conn_01x04_Socket, SW1 SW_DPDT, SW10 SW_DPDT, SW11 SW_DPDT, SW12 SW_DPDT, SW13 SW_DPDT, SW14 SW_DPDT, SW15 SW_DPDT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

Commit message: Write the soldering section.
Parts:
- J1: Alt Link (none) -> https://www.digikey.com/en/products/detail/w%C3%BCrth-elekt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
Changed lines of the file:
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@@
 			)
 		)
-		(property "Alt Link" ""
+		(property "Alt Link" "https://www.digikey.com/en/products/detail/w%C3%BCrth-elektronik/61202021621/2060592"
 			(at 140.97 142.24 0)
 			(effects
