File: PCBs/PerceptronInput/PerceptronInput.kicad_pcb (KiCad board)
At the start: 2 copper layers, 164 x 86 mm, 54 parts, among them J1 Conn_02x10, J2 Conn_01x04_Pin, SW1 SW_DPDT, SW10 SW_DPDT, SW11 SW_DPDT, SW12 SW_DPDT, SW13 SW_DPDT, SW14 SW_DPDT, SW15 SW_DPDT, SW16 SW_DPDT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

Commit message: Added resistor values to silkscreen.
Parts:
- R1, R10, R11, R12, R13, R14, R15, R16, R2, R3, R4, R5, R6, R7, R8, R9: footprint Resistor_THT:R_Axial_DIN0207_L6.3mm_D2.5mm_P7.62mm_Horizontal -> PerceptronInputFootprints:R_Axial_DIN0207_L6.3mm_D2.5mm_P7.62mm_Horizontal
Changed lines of the file:
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@@
 	(title_block
 		(title "Perceptron Input")
-		(date "2026-03-11")
-		(rev "2.2")
+		(date "2026-05-21")
+		(rev "2.3")
 		(company "RDB64")
 	)
@@
 		)
 	)
-	(footprint "Resistor_THT:R_Axial_DIN0207_L6.3mm_D2.5mm_P7.62mm_Horizontal"
+	(footprint "PerceptronInputFootprints:R_Axial_DIN0207_L6.3mm_D2.5mm_P7.62mm_Horizontal"
 		(layer "B.Cu")
 		(at 203 82.13 -90)
@@
 			(layer "B.Fab")
 		)
+		(fp_text user "${Value}"
+			(at 3.81 0 90)
+			(unlocked yes)
+			(layer "B.SilkS")
+			(effects
+				(font
+					(size 1 1)
+					(thickness 0.1)
+				)
+				(justify mirror)
+			)
+		)
 		(fp_text user "${REFERENCE}"
 			(at 3.81 0 90)
@@
 		)
 	)
-	(footprint "Resistor_THT:R_Axial_DIN0207_L6.3mm_D2.5mm_P7.62mm_Horizontal"
+	(footprint "PerceptronInputFootprints:R_Axial_DIN0207_L6.3mm_D2.5mm_P7.62mm_Horizontal"
 		(layer "B.Cu")
 		(at 187 82.13 -90)
@@
 			(layer "B.Fab")
 		)
+		(fp_text user "${Value}"
+			(at 3.81 0 90)
+			(unlocked yes)
+			(layer "B.SilkS")
+			(effects
+				(font
+					(size 1 1)
+					(thickness 0.1)
+				)
+				(justify mirror)
+			)
+		)
 		(fp_text user "${REFERENCE}"
 			(at 3.81 0 90)
@@
 		)
 	)
-	(footprint "Resistor_THT:R_Axial_DIN0207_L6.3mm_D2.5mm_P7.62mm_Horizontal"
+	(footprint "PerceptronInputFootprints:R_Axial_DIN0207_L6.3mm_D2.5mm_P7.62mm_Horizontal"
 		(layer "B.Cu")
 		(at 155 114.19 -90)
@@
 			(layer "B.Fab")
 		)
+		(fp_text user "${Value}"
+			(at 3.81 0 90)
+			(unlocked yes)
+			(layer "B.SilkS")
+			(effects
+				(font
+					(size 1 1)
+					(thickness 0.1)
+				)
+				(justify mirror)
+			)
+		)
 		(fp_text user "${REFERENCE}"
 			(at 3.81 0 90)
@@
 		)
 	)
-	(footprint "Resistor_THT:R_Axial_DIN0207_L6.3mm_D2.5mm_P7.62mm_Horizontal"
+	(footprint "PerceptronInputFootprints:R_Axial_DIN0207_L6.3mm_D2.5mm_P7.62mm_Horizontal"
 		(layer "B.Cu")
 		(at 187 98.19 -90)
@@
 			(layer "B.Fab")
 		)
+		(fp_text user "${Value}"
+			(at 3.81 0 90)
+			(unlocked yes)
+			(layer "B.SilkS")
+			(effects
+				(font
+					(size 1 1)
+					(thickness 0.1)
+				)
+				(justify mirror)
+			)
+		)
 		(fp_text user "${REFERENCE}"
 			(at 3.81 0 90)
@@
 			)
 		)
-		(property "Alt Link" ""
+		(property "Alt Link" "https://www.digikey.com/en/products/detail/w%C3%BCrth-elektronik/61202021621/2060592"
 			(at 0 0 180)
 			(unlocked yes)
@@
 		)
 	)
-	(footprint "Resistor_THT:R_Axial_DIN0207_L6.3mm_D2.5mm_P7.62mm_Horizontal"
+	(footprint "PerceptronInputFootprints:R_Axial_DIN0207_L6.3mm_D2.5mm_P7.62mm_Horizontal"
 		(layer "B.Cu")
 		(at 203 130.19 -90)
@@
 			(layer "B.Fab")
 		)
+		(fp_text user "${Value}"
+			(at 3.81 0 90)
+			(unlocked yes)
+			(layer "B.SilkS")
+			(effects
+				(font
+					(size 1 1)
+					(thickness 0.1)
+				)
+				(justify mirror)
+			)
+		)
 		(fp_text user "${REFERENCE}"
 			(at 3.81 0 90)
@@
 		)
 	)
-	(footprint "Resistor_THT:R_Axial_DIN0207_L6.3mm_D2.5mm_P7.62mm_Horizontal"
+	(footprint "PerceptronInputFootprints:R_Axial_DIN0207_L6.3mm_D2.5mm_P7.62mm_Horizontal"
 		(layer "B.Cu")
 		(at 171 114.19 -90)
@@
 			(layer "B.Fab")
 		)
+		(fp_text user "${Value}"
+			(at 3.81 0 90)
+			(unlocked yes)
+			(layer "B.SilkS")
+			(effects
+				(font
+					(size 1 1)
+					(thickness 0.1)
+				)
+				(justify mirror)
+			)
+		)
 		(fp_text user "${REFERENCE}"
 			(at 3.81 0 90)
@@
 		)
 	)
-	(footprint "Resistor_THT:R_Axial_DIN0207_L6.3mm_D2.5mm_P7.62mm_Horizontal"
+	(footprint "PerceptronInputFootprints:R_Axial_DIN0207_L6.3mm_D2.5mm_P7.62mm_Horizontal"
 		(layer "B.Cu")
 		(at 203 114.19 -90)
@@
 			(layer "B.Fab")
 		)
+		(fp_text user "${Value}"
+			(at 3.81 0 90)
+			(unlocked yes)
+			(layer "B.SilkS")
+			(effects
+				(font
+					(size 1 1)
+					(thickness 0.1)
+				)
+				(justify mirror)
+			)
+		)
 		(fp_text user "${REFERENCE}"
 			(at 3.81 0 90)
@@
 		)
 	)
-	(footprint "Resistor_THT:R_Axial_DIN0207_L6.3mm_D2.5mm_P7.62mm_Horizontal"
+	(footprint "PerceptronInputFootprints:R_Axial_DIN0207_L6.3mm_D2.5mm_P7.62mm_Horizontal"
 		(layer "B.Cu")
 		(at 203 98.19 -90)
@@
 			(layer "B.Fab")
 		)
+		(fp_text user "${Value}"
+			(at 3.81 0 90)
+			(unlocked yes)
+			(layer "B.SilkS")
+			(effects
+				(font
+					(size 1 1)
+					(thickness 0.1)
+				)
+				(justify mirror)
+			)
+		)
 		(fp_text user "${REFERENCE}"
 			(at 3.81 0 90)
@@
 		)
 	)
-	(footprint "Resistor_THT:R_Axial_DIN0207_L6.3mm_D2.5mm_P7.62mm_Horizontal"
+	(footprint "PerceptronInputFootprints:R_Axial_DIN0207_L6.3mm_D2.5mm_P7.62mm_Horizontal"
 		(layer "B.Cu")
 		(at 171 130.19 -90)
@@
 			(layer "B.Fab")
 		)
+		(fp_text user "${Value}"
+			(at 3.81 0 90)
+			(unlocked yes)
+			(layer "B.SilkS")
+			(effects
+				(font
+					(size 1 1)
+					(thickness 0.1)
+				)
+				(justify mirror)
+			)
+		)
 		(fp_text user "${REFERENCE}"
 			(at 3.81 0 90)
@@
 		)
 	)
-	(footprint "Resistor_THT:R_Axial_DIN0207_L6.3mm_D2.5mm_P7.62mm_Horizontal"
+	(footprint "PerceptronInputFootprints:R_Axial_DIN0207_L6.3mm_D2.5mm_P7.62mm_Horizontal"
 		(layer "B.Cu")
 		(at 187 114.19 -90)
@@
 			(layer "B.Fab")
 		)
+		(fp_text user "${Value}"
+			(at 3.81 0 90)
+			(unlocked yes)
+			(layer "B.SilkS")
+			(effects
+				(font
+					(size 1 1)
+					(thickness 0.1)
+				)
+				(justify mirror)
+			)
+		)
 		(fp_text user "${REFERENCE}"
 			(at 3.81 0 90)
@@
 		)
 	)
-	(footprint "Resistor_THT:R_Axial_DIN0207_L6.3mm_D2.5mm_P7.62mm_Horizontal"
+	(footprint "PerceptronInputFootprints:R_Axial_DIN0207_L6.3mm_D2.5mm_P7.62mm_Horizontal"
 		(layer "B.Cu")
 		(at 155 130.19 -90)
@@
 			(layer "B.Fab")
 		)
+		(fp_text user "${Value}"
+			(at 3.81 0 90)
+			(unlocked yes)
+			(layer "B.SilkS")
+			(effects
+				(font
+					(size 1 1)
+					(thickness 0.1)
+				)
+				(justify mirror)
+			)
+		)
 		(fp_text user "${REFERENCE}"
 			(at 3.81 0 90)
@@
 		)
 	)
-	(footprint "Resistor_THT:R_Axial_DIN0207_L6.3mm_D2.5mm_P7.62mm_Horizontal"
+	(footprint "PerceptronInputFootprints:R_Axial_DIN0207_L6.3mm_D2.5mm_P7.62mm_Horizontal"
 		(layer "B.Cu")
 		(at 155 98.19 -90)
@@
 			(layer "B.Fab")
 		)
+		(fp_text user "${Value}"
+			(at 3.81 0 90)
+			(unlocked yes)
+			(layer "B.SilkS")
+			(effects
+				(font
+					(size 1 1)
+					(thickness 0.1)
+				)
+				(justify mirror)
+			)
+		)
 		(fp_text user "${REFERENCE}"
 			(at 3.81 0 90)
@@
 		)
 	)
-	(footprint "Resistor_THT:R_Axial_DIN0207_L6.3mm_D2.5mm_P7.62mm_Horizontal"
+	(footprint "PerceptronInputFootprints:R_Axial_DIN0207_L6.3mm_D2.5mm_P7.62mm_Horizontal"
 		(layer "B.Cu")
 		(at 171 82.13 -90)
@@
 			(layer "B.Fab")
 		)
+		(fp_text user "${Value}"
+			(at 3.81 0 90)
+			(unlocked yes)
+			(layer "B.SilkS")
+			(effects
+				(font
+					(size 1 1)
+					(thickness 0.1)
+				)
+				(justify mirror)
+			)
+		)
 		(fp_text user "${REFERENCE}"
 			(at 3.81 0 90)
@@
 		)
 	)
-	(footprint "Resistor_THT:R_Axial_DIN0207_L6.3mm_D2.5mm_P7.62mm_Horizontal"
+	(footprint "PerceptronInputFootprints:R_Axial_DIN0207_L6.3mm_D2.5mm_P7.62mm_Horizontal"
 		(layer "B.Cu")
 		(at 155 82.13 -90)
@@
 			(layer "B.Fab")
 		)
+		(fp_text user "${Value}"
+			(at 3.81 0 90)
+			(unlocked yes)
+			(layer "B.SilkS")
+			(effects
+				(font
+					(size 1 1)
+					(thickness 0.1)
+				)
+				(justify mirror)
+			)
+		)
 		(fp_text user "${REFERENCE}"
 			(at 3.81 0 90)
@@
 		)
 	)
-	(footprint "Resistor_THT:R_Axial_DIN0207_L6.3mm_D2.5mm_P7.62mm_Horizontal"
+	(footprint "PerceptronInputFootprints:R_Axial_DIN0207_L6.3mm_D2.5mm_P7.62mm_Horizontal"
 		(layer "B.Cu")
 		(at 187 130.19 -90)
@@
 			(layer "B.Fab")
 		)
+		(fp_text user "${Value}"
+			(at 3.81 0 90)
+			(unlocked yes)
+			(layer "B.SilkS")
+			(effects
+				(font
+					(size 1 1)
+					(thickness 0.1)
+				)
+				(justify mirror)
+			)
+		)
 		(fp_text user "${REFERENCE}"
 			(at 3.81 0 90)
@@
 		)
 	)
-	(footprint "Resistor_THT:R_Axial_DIN0207_L6.3mm_D2.5mm_P7.62mm_Horizontal"
+	(footprint "PerceptronInputFootprints:R_Axial_DIN0207_L6.3mm_D2.5mm_P7.62mm_Horizontal"
 		(layer "B.Cu")
 		(at 171 98.19 -90)
@@
 			(layer "B.Fab")
 		)
+		(fp_text user "${Value}"
+			(at 3.81 0 90)
+			(unlocked yes)
+			(layer "B.SilkS")
+			(effects
+				(font
+					(size 1 1)
+					(thickness 0.1)
+				)
+				(justify mirror)
+			)
+		)
 		(fp_text user "${REFERENCE}"
